File: deska.brd (EAGLE design)
At the start: 64.4 x 69.8 mm, 17 parts, among them X1 JST-XH-03-PIN-LONG-PAD

Commit message: +
Parts:
- removed I2C, I2C1: JST-XH-04-PIN-LONG-PAD, Rembrandt Electronics - JST XH Connectors v1-0:JST-XH-04-PACKAGE-LONG-PAD
- removed IN, OUT, RADIATORS, SERIAL, X1: JST-XH-03-PIN-LONG-PAD, Rembrandt Electronics - JST XH Connectors v1-0:JST-XH-03-PACKAGE-LONG-PAD
- removed SOURCE: (no value), con-wago-508:W237-132
- added BUZZER, NAPAJENI: (no value), con-wago-508:W237-132
- added I2CDISP, I2CKEYB: (no value), con-wago-508:W237-4P
- added Q1: BC547, transistor-npn:TO92
- added R6: 1k, rcl:0207/7
- added TIN, TOUT, TUT: (no value), con-wago-508:W237-3E
- LED: value JST-XH-02-PIN-LONG-PAD -> (none); device Rembrandt Electronics - JST XH Connectors v1-0:JST-XH-02-PACKAGE-LONG-PAD -> con-wago-508:W237-132
- LED1: device led:LED3MM -> con-wago-508:W237-132
- R1, R3, R5: device rcl:0207/10 -> rcl:0207/7
- R2: value 220 -> 4k7; device rcl:0207/10 -> rcl:0207/7
- R4: value 4k7 -> 220; device rcl:0207/10 -> rcl:0207/7
- RELAY: value JST-XH-03-PIN-LONG-PAD -> (none); device Rembrandt Electronics - JST XH Connectors v1-0:JST-XH-03-PACKAGE-LONG-PAD -> con-wago-508:W237-132
- WEMOS1: device esp8266modules:WEMOS-D1-MINI -> wemos:WEMOS-D1-MINI
- moved R4 77.3 mm to (88.9, 53.3), turned to 90 degrees
- moved LED 66.5 mm to (64.8, 68.6)
- moved LED1 46.2 mm to (-6.35, 7.62)
- moved RELAY 41.3 mm to (53.3, 68.6), turned to 0 degrees
- moved R1 37.9 mm to (21.6, 52.1)
- moved R5 37.2 mm to (-6.35, -3.81)
- moved WEMOS1 19.1 mm to (44.5, 36.8)
- moved R2 14.8 mm to (21.6, 33.0), turned to 180 degrees
- moved R3 8.13 mm to (21.6, 12.7)
Connections:
- removed net N$10: LED1.A, R5.2
- removed net N$13: OUT.1, R3.2, WEMOS1.D6
- removed net N$4: I2C.3, I2C1.3, WEMOS1.D2
- removed net N$9: IN.1, R4.2, WEMOS1.D7
- new net N$12: I2CDISP.3, I2CKEYB.3, WEMOS1.D2
- new net N$14: R5.1, RELAY.1, WEMOS1.D3
- new net N$15: BUZZER.1, Q1.3
- new net N$19: R2.1, TOUT.3, WEMOS1.D5
- net +5V: now also I2CDISP.2, I2CKEYB.2, LED.2, LED1.1, NAPAJENI.1, R1.2, R2.2, R3.2, RELAY.2, TIN.2, TOUT.2, TUT.2; no longer I2C.2, I2C1.2, IN.2, LED.1, OUT.2, R1.1, R3.1, R4.1, R5.1, RADIATORS.2, RELAY.3, SOURCE.1, X1.3
- net GND: now also BUZZER.2, I2CDISP.1, I2CKEYB.1, NAPAJENI.2, Q1.1, TIN.1, TOUT.1, TUT.1; no longer I2C.1, I2C1.1, IN.3, LED1.K, OUT.3, RADIATORS.3, RELAY.2, SERIAL.1, SOURCE.2, X1.1
- net N$1: now also R1.1, TIN.3, WEMOS1.D0; no longer SERIAL.2, WEMOS1.TX
- net N$11: now also I2CDISP.4, I2CKEYB.4, WEMOS1.D1; no longer R1.2, RADIATORS.1, WEMOS1.D5
- net N$2: now also LED1.2, R5.2; no longer SERIAL.3, WEMOS1.RX
- net N$3: now also R3.1, TUT.3, WEMOS1.D6; no longer I2C.4, I2C1.4, WEMOS1.D1
- net N$5: now also R4.1, WEMOS1.D8; no longer WEMOS1.D0, X1.2
- net N$6: now also LED.1, R4.2; no longer R2.1, WEMOS1.D4
- net N$7: now also Q1.2, R6.1; no longer RELAY.1, WEMOS1.D3
- net N$8: now also R6.2, WEMOS1.D7; no longer LED.2, R2.2
Routing:
- net GND: track 217.3 -> 53.3 mm
- net +5V: track 169.6 -> 73.7 mm
- net N$4: track 49.5 -> 0.00 mm
- net N$11: track 34.7 -> 0.00 mm
- net N$9: track 31.1 -> 0.00 mm
- net N$13: track 28.2 -> 0.00 mm
- net N$19: track 0.00 -> 20.5 mm
- net N$1: track 7.62 -> 27.4 mm
- net N$3: track 49.5 -> 32.2 mm
- net N$5: track 12.8 -> 0.00 mm
- net N$8: track 12.5 -> 0.00 mm
- net N$7: track 8.67 -> 0.00 mm
- net N$2: track 7.62 -> 0.00 mm
- net N$6: track 3.81 -> 0.00 mm
- net N$10: track 2.54 -> 0.00 mm
Other:
- board size 64.4 x 69.8 mm -> 100 x 80 mm

Commit message: +
Connections:
- new net BUILTINLED: WEMOS1.D4
Changed lines of the file:
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@@
 <wire x1="34.29" y1="31.75" x2="90.17" y2="63.5" width="0" layer="19" extent="1-1"/>
+</signal>
+<signal name="BUILTINLED">
+<contactref element="WEMOS1" pad="D4"/>
 </signal>
 </signals>

Commit message: upravy kodu
Parts:
- removed I2CDISP, I2CKEYB: (no value), con-wago-508:W237-4P
- removed LED: (no value), con-wago-508:W237-132
- removed TIN, TOUT, TUT: (no value), con-wago-508:W237-3E
- added LEDRELAY: JST-XH-02-PIN-LONG-PAD, Rembrandt Electronics - JST XH Connectors v1-0:JST-XH-02-PACKAGE-LONG-PAD
- added X1, X2, X3: JST-XH-03-PIN-LONG-PAD, Rembrandt Electronics - JST XH Connectors v1-0:JST-XH-03-PACKAGE-LONG-PAD
- added X4, X5, X6: JST-XH-04-PIN-LONG-PAD, Rembrandt Electronics - JST XH Connectors v1-0:JST-XH-04-PACKAGE-LONG-PAD
- BUZZER, LED1: value (none) -> JST-XH-02-PIN-LONG-PAD; device con-wago-508:W237-132 -> Rembrandt Electronics - JST XH Connectors v1-0:JST-XH-02-PACKAGE-LONG-PAD
- RELAY: value (none) -> JST-XH-03-PIN-LONG-PAD; device con-wago-508:W237-132 -> Rembrandt Electronics - JST XH Connectors v1-0:JST-XH-03-PACKAGE-LONG-PAD
- moved R5 65.6 mm to (49.5, 30.5), turned to 270 degrees
- moved NAPAJENI 58.5 mm to (72.4, 17.8)
- moved R4 56.9 mm to (39.4, 25.4), turned to 270 degrees
- moved RELAY 55.9 mm to (55.9, 12.7)
- moved R6 54.7 mm to (39.4, 35.6), turned to 270 degrees
- moved LED1 36.1 mm to (29.2, 14.0), turned to 90 degrees
- moved Q1 29.3 mm to (63.5, 47.0), turned to 90 degrees
- moved BUZZER 26.2 mm to (71.1, 48.3), turned to 180 degrees
- moved R1 11.5 mm to (22.9, 40.6)
- moved R3 10.2 mm to (22.9, 22.9)
- moved R2 1.80 mm to (22.9, 31.8)
Connections:
- new net +3V3: LED1.2, LEDRELAY.2, R1.2, R2.2, R3.2, WEMOS1.3V3, X1.2, X2.2, X3.2
- new net N$9: WEMOS1.GND, X4.3, X5.3, X6.3
- net +5V: now also BUZZER.1, X4.4, X5.4, X6.4; no longer I2CDISP.2, I2CKEYB.2, LED.2, LED1.1, R1.2, R2.2, R3.2, TIN.2, TOUT.2, TUT.2
- net GND: now also RELAY.3, X1.3, X2.3, X3.3; no longer BUZZER.2, I2CDISP.1, I2CKEYB.1, TIN.1, TOUT.1, TUT.1, WEMOS1.GND
- net N$1: now also X1.1; no longer TIN.3
- net N$11: now also X4.1, X5.1, X6.1; no longer I2CDISP.4, I2CKEYB.4
- net N$12: now also X4.2, X5.2, X6.2; no longer I2CDISP.3, I2CKEYB.3
- net N$15: now also BUZZER.2; no longer BUZZER.1
- net N$19: now also X2.1; no longer TOUT.3
- net N$2: now also LEDRELAY.1; no longer LED1.2
- net N$3: now also X3.1; no longer TUT.3
- net N$6: now also LED1.1; no longer LED.1
Routing:
- net GND: track 53.3 -> 166.1 mm
- net +3V3: track 0.00 -> 76.6 mm
- net N$2: track 0.00 -> 40.5 mm
- net N$14: track 0.00 -> 29.3 mm
- net N$7: track 0.00 -> 26.9 mm
- net N$9: track 0.00 -> 25.4 mm
- net N$12: track 0.00 -> 20.3 mm
- net N$11: track 0.00 -> 20.3 mm
- net N$6: track 0.00 -> 16.8 mm
- net N$3: track 32.2 -> 16.8 mm
- net N$1: track 27.4 -> 13.2 mm, vias 0 -> 1
- net N$19: track 20.5 -> 12.7 mm
- net N$15: track 0.00 -> 7.40 mm
- net N$8: track 0.00 -> 5.08 mm
- net N$5: track 0.00 -> 5.08 mm
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Other:
- board size 100 x 80 mm -> 72.1 x 55.9 mm
