File: deska.sch (EAGLE design)
At the start: 23 parts, among them Q1 BC547, X1 JST-XH-03-PIN-LONG-PAD, X2 JST-XH-03-PIN-LONG-PAD, X3 JST-XH-03-PIN-LONG-PAD, X4 JST-XH-04-PIN-LONG-PAD, X5 JST-XH-04-PIN-LONG-PAD, X6 JST-XH-04-PIN-LONG-PAD, X7 JST-XH-03-PIN-LONG-PAD

Commit message: +
Connections:
- removed net N$3: WEMOS1.D8, X7-3.S
- new net N$10: WEMOS1.D0, X7-3.S
- net N$8: now also WEMOS1.D8; no longer WEMOS1.D0
Other:
- moved on the sheet: BUZZER-1, BUZZER-2, Q1, R6
Changed lines of the file:
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@@
 <attribute name="VALUE" x="24.13" y="41.402" size="1.778" layer="96" rot="R180"/>
 </instance>
-<instance part="Q1" gate="G$1" x="129.54" y="40.64" smashed="yes">
-<attribute name="NAME" x="119.38" y="48.26" size="1.778" layer="95"/>
-<attribute name="VALUE" x="119.38" y="45.72" size="1.778" layer="96"/>
-</instance>
-<instance part="R6" gate="G$1" x="121.92" y="40.64" smashed="yes" rot="R180">
-<attribute name="NAME" x="125.73" y="39.1414" size="1.778" layer="95" rot="R180"/>
-<attribute name="VALUE" x="125.73" y="43.942" size="1.778" layer="96" rot="R180"/>
+<instance part="Q1" gate="G$1" x="121.92" y="40.64" smashed="yes">
+<attribute name="NAME" x="111.76" y="48.26" size="1.778" layer="95"/>
+<attribute name="VALUE" x="111.76" y="45.72" size="1.778" layer="96"/>
+</instance>
+<instance part="R6" gate="G$1" x="106.68" y="40.64" smashed="yes" rot="R180">
+<attribute name="NAME" x="110.49" y="39.1414" size="1.778" layer="95" rot="R180"/>
+<attribute name="VALUE" x="110.49" y="43.942" size="1.778" layer="96" rot="R180"/>
 </instance>
 <instance part="P+1" gate="1" x="-12.7" y="53.34" smashed="yes" rot="R270">
 <attribute name="VALUE" x="-17.78" y="55.88" size="1.778" layer="96"/>
 </instance>
-<instance part="GND4" gate="1" x="132.08" y="30.48" smashed="yes">
-<attribute name="VALUE" x="129.54" y="27.94" size="1.778" layer="96"/>
+<instance part="GND4" gate="1" x="124.46" y="30.48" smashed="yes">
+<attribute name="VALUE" x="121.92" y="27.94" size="1.778" layer="96"/>
 </instance>
 <instance part="GND5" gate="1" x="0" y="50.8" smashed="yes">
@@
 <attribute name="VALUE" x="14.097" y="8.382" size="1.778" layer="96" rot="R270"/>
 </instance>
-<instance part="BUZZER" gate="-2" x="134.62" y="58.42" smashed="yes">
-<attribute name="NAME" x="137.16" y="57.658" size="1.524" layer="95"/>
-</instance>
-<instance part="BUZZER" gate="-1" x="134.62" y="60.96" smashed="yes">
-<attribute name="NAME" x="137.16" y="60.198" size="1.524" layer="95"/>
-<attribute name="VALUE" x="133.858" y="62.357" size="1.778" layer="96"/>
+<instance part="BUZZER" gate="-2" x="127" y="58.42" smashed="yes">
+<attribute name="NAME" x="129.54" y="57.658" size="1.524" layer="95"/>
+</instance>
+<instance part="BUZZER" gate="-1" x="129.54" y="60.96" smashed="yes">
+<attribute name="NAME" x="132.08" y="60.198" size="1.524" layer="95"/>
+<attribute name="VALUE" x="128.778" y="62.357" size="1.778" layer="96"/>
 </instance>
 <instance part="P+2" gate="1" x="106.68" y="58.42" smashed="yes">
@@
 <pinref part="Q1" gate="G$1" pin="E"/>
 <pinref part="GND4" gate="1" pin="GND"/>
-<wire x1="132.08" y1="35.56" x2="132.08" y2="33.02" width="0.1524" layer="91"/>
+<wire x1="124.46" y1="35.56" x2="124.46" y2="33.02" width="0.1524" layer="91"/>
 </segment>
 <segment>
@@
 <segment>
 <wire x1="111.76" y1="73.66" x2="129.54" y2="73.66" width="0.1524" layer="91"/>
-<wire x1="111.76" y1="73.66" x2="93.98" y2="73.66" width="0.1524" layer="91"/>
+<wire x1="111.76" y1="73.66" x2="88.9" y2="73.66" width="0.1524" layer="91"/>
 <junction x="111.76" y="73.66"/>
 <pinref part="WEMOS1" gate="D1" pin="D2"/>
-<wire x1="81.28" y1="63.5" x2="93.98" y2="63.5" width="0.1524" layer="91"/>
-<wire x1="93.98" y1="63.5" x2="93.98" y2="73.66" width="0.1524" layer="91"/>
+<wire x1="81.28" y1="63.5" x2="88.9" y2="63.5" width="0.1524" layer="91"/>
+<wire x1="88.9" y1="63.5" x2="88.9" y2="73.66" width="0.1524" layer="91"/>
 <pinref part="X4" gate="-2" pin="S"/>
 <wire x1="111.76" y1="78.74" x2="111.76" y2="73.66" width="0.1524" layer="91"/>
@@
 <segment>
 <wire x1="109.22" y1="76.2" x2="127" y2="76.2" width="0.1524" layer="91"/>
-<wire x1="109.22" y1="76.2" x2="91.44" y2="76.2" width="0.1524" layer="91"/>
+<wire x1="109.22" y1="76.2" x2="86.36" y2="76.2" width="0.1524" layer="91"/>
 <junction x="109.22" y="76.2"/>
 <pinref part="WEMOS1" gate="D1" pin="D1"/>
-<wire x1="81.28" y1="66.04" x2="91.44" y2="66.04" width="0.1524" layer="91"/>
-<wire x1="91.44" y1="66.04" x2="91.44" y2="76.2" width="0.1524" layer="91"/>
+<wire x1="81.28" y1="66.04" x2="86.36" y2="66.04" width="0.1524" layer="91"/>
+<wire x1="86.36" y1="66.04" x2="86.36" y2="76.2" width="0.1524" layer="91"/>
 <pinref part="X4" gate="-1" pin="S"/>
 <wire x1="109.22" y1="78.74" x2="109.22" y2="76.2" width="0.1524" layer="91"/>
@@
 <wire x1="-25.4" y1="43.18" x2="35.56" y2="43.18" width="0.1524" layer="91"/>
 <pinref part="WEMOS1" gate="D1" pin="D3"/>
-<wire x1="35.56" y1="43.18" x2="93.98" y2="43.18" width="0.1524" layer="91"/>
-<wire x1="93.98" y1="43.18" x2="93.98" y2="60.96" width="0.1524" layer="91"/>
-<wire x1="93.98" y1="60.96" x2="81.28" y2="60.96" width="0.1524" layer="91"/>
+<wire x1="35.56" y1="43.18" x2="88.9" y2="43.18" width="0.1524" layer="91"/>
+<wire x1="88.9" y1="43.18" x2="88.9" y2="60.96" width="0.1524" layer="91"/>
+<wire x1="88.9" y1="60.96" x2="81.28" y2="60.96" width="0.1524" layer="91"/>
 <pinref part="R5" gate="G$1" pin="1"/>
 <wire x1="35.56" y1="17.78" x2="25.4" y2="17.78" width="0.1524" layer="91"/>
@@
 <segment>
 <pinref part="Q1" gate="G$1" pin="C"/>
-<wire x1="132.08" y1="58.42" x2="132.08" y2="45.72" width="0.1524" layer="91"/>
+<wire x1="124.46" y1="58.42" x2="124.46" y2="45.72" width="0.1524" layer="91"/>
 <pinref part="BUZZER" gate="-2" pin="S"/>
 </segment>
@@
 </segment>
 <segment>
-<wire x1="124.46" y1="60.96" x2="132.08" y2="60.96" width="0.1524" layer="91"/>
+<wire x1="124.46" y1="60.96" x2="127" y2="60.96" width="0.1524" layer="91"/>
 <pinref part="WEMOS1" gate="D1" pin="5V"/>
 <wire x1="81.28" y1="53.34" x2="106.68" y2="53.34" width="0.1524" layer="91"/>
@@
 <pinref part="R6" gate="G$1" pin="1"/>
 <pinref part="Q1" gate="G$1" pin="B"/>
+<wire x1="111.76" y1="40.64" x2="119.38" y2="40.64" width="0.1524" layer="91"/>
 </segment>
 </net>
@@
 <net name="N$8" class="0">
 <segment>
-<pinref part="WEMOS1" gate="D1" pin="D0"/>
-<wire x1="48.26" y1="66.04" x2="45.72" y2="66.04" width="0.1524" layer="91"/>
 <pinref part="R6" gate="G$1" pin="2"/>
-<wire x1="45.72" y1="66.04" x2="45.72" y2="40.64" width="0.1524" layer="91"/>
-<wire x1="45.72" y1="40.64" x2="116.84" y2="40.64" width="0.1524" layer="91"/>
-</segment>
-</net>
-<net name="N$3" class="0">
-<segment>
+<wire x1="45.72" y1="40.64" x2="101.6" y2="40.64" width="0.1524" layer="91"/>
+<wire x1="45.72" y1="40.64" x2="45.72" y2="55.88" width="0.1524" layer="91"/>
 <pinref part="WEMOS1" gate="D1" pin="D8"/>
-<wire x1="48.26" y1="55.88" x2="40.64" y2="55.88" width="0.1524" layer="91"/>
-<wire x1="40.64" y1="17.78" x2="40.64" y2="55.88" width="0.1524" layer="91"/>
-<pinref part="X7" gate="-3" pin="S"/>
+<wire x1="45.72" y1="55.88" x2="48.26" y2="55.88" width="0.1524" layer="91"/>
 </segment>
 </net>
@@
 </segment>
 </net>
+<net name="N$10" class="0">
+<segment>
+<pinref part="WEMOS1" gate="D1" pin="D0"/>
+<wire x1="40.64" y1="17.78" x2="40.64" y2="66.04" width="0.1524" layer="91"/>
+<pinref part="X7" gate="-3" pin="S"/>
+<wire x1="48.26" y1="66.04" x2="40.64" y2="66.04" width="0.1524" layer="91"/>
+</segment>
+</net>

Commit message: +
Connections:
- net +3V3: no longer X7-2.S
- net +5V: now also X7-2.S
Changed lines of the file:
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@@
 <part name="LED2" library="led" library_urn="urn:adsk.eagle:library:259" deviceset="LED" device="3MM" package3d_urn="urn:adsk.eagle:package:15797/1" value="LED2"/>
 <part name="GND2" library="supply1" deviceset="GND" device=""/>
-<part name="+3V5" library="supply1" library_urn="urn:adsk.eagle:library:371" deviceset="+3V3" device=""/>
 <part name="X7" library="Rembrandt Electronics - JST XH Connectors v1-0" deviceset="JST-XH-03-PIN" device="-LONG-PAD"/>
 <part name="GND3" library="supply1" deviceset="GND" device=""/>
 <part name="RESET" library="Rembrandt Electronics - JST XH Connectors v1-0" deviceset="JST-XH-02-PIN" device="-LONG-PAD"/>
 <part name="GND7" library="supply1" deviceset="GND" device=""/>
+<part name="P+3" library="supply1" deviceset="+5V" device=""/>
 </parts>
 <sheets>
@@
 <attribute name="VALUE" x="101.6" y="66.04" size="1.778" layer="96"/>
 </instance>
-<instance part="+3V5" gate="G$1" x="43.18" y="25.4" smashed="yes">
-<attribute name="VALUE" x="40.64" y="20.32" size="1.778" layer="96" rot="R90"/>
-</instance>
 <instance part="X7" gate="-1" x="45.72" y="15.24" smashed="yes" rot="R270">
 <attribute name="NAME" x="44.958" y="12.7" size="1.524" layer="95" rot="R270"/>
@@
 <instance part="GND7" gate="1" x="43.18" y="73.66" smashed="yes">
 <attribute name="VALUE" x="40.64" y="71.12" size="1.778" layer="96"/>
+</instance>
+<instance part="P+3" gate="1" x="43.18" y="25.4" smashed="yes">
+<attribute name="VALUE" x="40.64" y="20.32" size="1.778" layer="96" rot="R90"/>
 </instance>
 </instances>
@@
 <wire x1="106.68" y1="55.88" x2="106.68" y2="53.34" width="0.1524" layer="91"/>
 <junction x="106.68" y="53.34"/>
+</segment>
+<segment>
+<wire x1="43.18" y1="22.86" x2="43.18" y2="17.78" width="0.1524" layer="91"/>
+<pinref part="X7" gate="-2" pin="S"/>
+<pinref part="P+3" gate="1" pin="+5V"/>
 </segment>
 </net>
@@
 <pinref part="X3" gate="-2" pin="S"/>
 </segment>
-<segment>
-<pinref part="+3V5" gate="G$1" pin="+3V3"/>
-<wire x1="43.18" y1="22.86" x2="43.18" y2="17.78" width="0.1524" layer="91"/>
-<pinref part="X7" gate="-2" pin="S"/>
-</segment>
-</net>
+</net>
